File: varLoad.sch (KiCad schematic (older format))
At the start: 15 parts, among them Q1 MTP3055, SW1 SPST, U1 LM324

Commit message: started placement
Parts:
- removed BT1: 4xAAA, ~, symbol BATTERY
- removed SW1: SPST, ~, symbol SPST
- added P1: CONN_2, symbol CONN_2
- added P2: V+, symbol CONN_1
- added P3: V-, symbol CONN_1
- C1: value C -> 0.1u
- R1: Part Number (none) -> P10.0KFCT-ND
- U1: Part Number (none) -> 296-1391-5-ND
Connections:
- net +6V: now also D2.2 (K)
- net GND: now also P1.2 (PM)
- net at D2.1 (A): now also P1.1 (P1)
Other:
- note removed: "Spec low voltage drop part."
- moved on the sheet: D2
Changed lines of the file:
@@
 Sheet 1 1
 Title ""
-Date "8 mar 2014"
+Date "10 mar 2014"
 Rev ""
 Comp ""
@@
 F 2 "" H 4550 3800 60  0000 C CNN
 F 3 "" H 4550 3800 60  0000 C CNN
+F 4 "296-1391-5-ND" H 4550 3800 60  0001 C CNN "Part Number"
 	1    4550 3800
 	1    0    0    -1
@@
 1060K-ND  NICE COIN CELL HOLDERS  - COULD USE 2 TO GET 6V
 $Comp
-L BATTERY BT1
-U 1 1 5302B749
-P 3450 1450
-F 0 "BT1" H 3450 1650 50  0000 C CNN
-F 1 "4xAAA" H 3450 1260 50  0000 C CNN
-F 2 "~" H 3450 1450 60  0000 C CNN
-F 3 "~" H 3450 1450 60  0000 C CNN
-F 4 "2481K-ND" H 3450 1450 60  0001 C CNN "Part Number"
-	1    3450 1450
-	1    0    0    -1
-$EndComp
-$Comp
 L GND #PWR011
 U 1 1 5302B766
-P 3950 1800
-F 0 "#PWR011" H 3950 1800 30  0001 C CNN
-F 1 "GND" H 3950 1730 30  0001 C CNN
-F 2 "" H 3950 1800 60  0000 C CNN
-F 3 "" H 3950 1800 60  0000 C CNN
-	1    3950 1800
+P 1700 1800
+F 0 "#PWR011" H 1700 1800 30  0001 C CNN
+F 1 "GND" H 1700 1730 30  0001 C CNN
+F 2 "" H 1700 1800 60  0000 C CNN
+F 3 "" H 1700 1800 60  0000 C CNN
+	1    1700 1800
 	1    0    0    -1
 $EndComp
@@
 L +6V #PWR012
 U 1 1 5302B76C
-P 1300 1200
-F 0 "#PWR012" H 1300 1290 20  0001 C CNN
-F 1 "+6V" H 1300 1290 30  0000 C CNN
-F 2 "" H 1300 1200 60  0000 C CNN
-F 3 "" H 1300 1200 60  0000 C CNN
-	1    1300 1200
-	1    0    0    -1
-$EndComp
-$Comp
-L SPST SW1
-U 1 1 5302B859
-P 1950 1450
-F 0 "SW1" H 1950 1550 70  0000 C CNN
-F 1 "SPST" H 1950 1350 70  0000 C CNN
-F 2 "~" H 1950 1450 60  0000 C CNN
-F 3 "~" H 1950 1450 60  0000 C CNN
-	1    1950 1450
-	-1   0    0    1
-$EndComp
-Wire Wire Line
-	2950 1450 3150 1450
-Wire Wire Line
-	1300 1450 1450 1450
+P 1700 1350
+F 0 "#PWR012" H 1700 1440 20  0001 C CNN
+F 1 "+6V" H 1700 1440 30  0000 C CNN
+F 2 "" H 1700 1350 60  0000 C CNN
+F 3 "" H 1700 1350 60  0000 C CNN
+	1    1700 1350
+	1    0    0    -1
+$EndComp
 $Comp
 L C C1
@@
 P 5850 2450
 F 0 "C1" H 5850 2550 40  0000 L CNN
-F 1 "C" H 5856 2365 40  0000 L CNN
+F 1 "0.1u" H 5856 2365 40  0000 L CNN
 F 2 "~" H 5888 2300 30  0000 C CNN
 F 3 "~" H 5850 2450 60  0000 C CNN
@@
 Wire Wire Line
 	5850 2250 5850 2150
-Connection ~ 3050 1450
 $Comp
 L DIODE D2
 U 1 1 5302BAA4
-P 2750 1450
-F 0 "D2" H 2750 1550 40  0000 C CNN
-F 1 "DIODE" H 2750 1350 40  0000 C CNN
-F 2 "~" H 2750 1450 60  0000 C CNN
-F 3 "~" H 2750 1450 60  0000 C CNN
-	1    2750 1450
+P 2100 1450
+F 0 "D2" H 2100 1550 40  0000 C CNN
+F 1 "DIODE" H 2100 1350 40  0000 C CNN
+F 2 "~" H 2100 1450 60  0000 C CNN
+F 3 "~" H 2100 1450 60  0000 C CNN
+	1    2100 1450
 	-1   0    0    1
 $EndComp
-Wire Wire Line
-	2550 1450 2450 1450
-Wire Wire Line
-	1300 1450 1300 1200
-Wire Wire Line
-	3950 1800 3950 1450
 $Comp
 L +6V #PWR015
@@
 F 2 "~" V 1730 3100 30  0000 C CNN
 F 3 "~" H 1800 3100 30  0000 C CNN
+F 4 "P10.0KFCT-ND" H 1800 3100 60  0001 C CNN "Part Number"
 	1    1800 3100
 	-1   0    0    1
@@
 Wire Wire Line
 	1800 3900 1800 4050
-Text Notes 2250 1850 0    60   ~ 0
-Spec low voltage drop part.
-Wire Wire Line
-	3950 1450 3750 1450
+$Comp
+L CONN_2 P1
+U 1 1 531C77E9
+P 3000 1550
+F 0 "P1" V 2950 1550 40  0000 C CNN
+F 1 "CONN_2" V 3050 1550 40  0000 C CNN
+F 2 "" H 3000 1550 60  0000 C CNN
+F 3 "" H 3000 1550 60  0000 C CNN
+F 4 "RASM722PX" H 3000 1550 60  0001 C CNN "Part Number"
+F 5 "Switch Craft" H 3000 1550 60  0001 C CNN "MFG Name"
+	1    3000 1550
+	1    0    0    -1
+$EndComp
+Wire Wire Line
+	2300 1450 2650 1450
+Wire Wire Line
+	1700 1800 1700 1650
+Wire Wire Line
+	1700 1650 2650 1650
+Wire Wire Line
+	1900 1450 1700 1450
+Wire Wire Line
+	1700 1450 1700 1350
+$Comp
+L CONN_1 P2
+U 1 1 531D156A
+P 9000 2500
+F 0 "P2" V 9000 2350 40  0000 L CNN
+F 1 "V+" H 9000 2555 30  0001 C CNN
+F 2 "" H 9000 2500 60  0000 C CNN
+F 3 "" H 9000 2500 60  0000 C CNN
+	1    9000 2500
+	0    -1   -1   0
+$EndComp
+$Comp
+L CONN_1 P3
+U 1 1 531D1579
+P 9000 3000
+F 0 "P3" V 9000 3050 40  0000 L CNN
+F 1 "V-" H 9000 3055 30  0001 C CNN
+F 2 "" H 9000 3000 60  0000 C CNN
+F 3 "" H 9000 3000 60  0000 C CNN
+	1    9000 3000
+	0    1    1    0
+$EndComp
 $EndSCHEMATC
